File: Kicad/MacroPadV2.kicad_sch (KiCad schematic)
At the start: 26 parts, among them K1 KSW, K10 KSW, K11 KSW, K12 KSW, K2 KSW, K3 KSW, K4 KSW, K5 KSW, K6 KSW, K7 KSW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

Commit message: Started V2 	-More space between keys(keycaps didnt fit) 	-Pull Down Resistors for Columns and Rotary Switch(ATMega32U4 is internal pull up) 	-Slightly larger board and edge holes
Parts:
- added R1, R2, R3, R4, R5: 1k, Resistor_SMD:R_0805_2012Metric_Pad1.20x1.40mm_HandSolder, symbol Device:R_Small_US
- D1, D10, D11, D12, D2, D3, D4, D5, D6, D7, D8, D9: footprint aarohanl:CR_SOD323_MCC-L -> mpadfps:sod323
Connections:
- net COL0: now also R1.1
- net COL1: now also R2.1
- net COL2: now also R3.1
- net COL3: now also R4.1
- net GND: now also R1.2, R2.2, R3.2, R4.2, R5.2
- net PD4: now also R5.1
